File: xl_maxsonar_adapter.kicad_pcb (KiCad board)
At the start: 2 copper layers, 20 x 19.2 mm, 2 parts, among them J1 Conn_01x07, J2 Conn_01x04

Commit message: Added R2 to silkscreen. Made new gerber files.
Other:
- board text added: "XL MaxSonar Adapter v0.1 R2 www.iorodeo.com"
- board text removed: "XL MaxSonar Adapter v0.1 www.iorodeo.com"
Changed lines of the file:
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@@
       (drillshape 0)
       (scaleselection 1)
-      (outputdirectory "production/v0p1_r1/gerber/")
+      (outputdirectory "production/v0p1_r2/gerber/")
     )
   )
@@
   (gr_line (start 58 65.8) (end 58 68.25)
     (stroke (width 0.2) (type default)) (layer "Edge.Cuts"))
-  (gr_text "XL MaxSonar \nAdapter v0.1\nwww.iorodeo.com" (at 54.2 59.3 270) (layer "B.SilkS")
+  (gr_text "XL MaxSonar \nAdapter v0.1 R2\nwww.iorodeo.com" (at 54.1 59.3 270) (layer "B.SilkS")
     (effects (font (size 1 1) (thickness 0.15)) (justify bottom mirror))
   )
